Commit message: turn on spot depth cameras
add qr code detection using qreader
add motion detection node
and few more changes

File: spot_driver_plus/urdf/gen3.urdf.xacro (robot description, xacro)
@@ -70,5 +70,5 @@
     <child link="front_collision" />
     <parent link="body" />
-    <origin xyz="0.35 0 0.15" rpy="0 0 0" />
+    <origin xyz="0.3 0 0.15" rpy="0 0 0" />
   </joint>
   <!-- Back CB -->
